File: hardware/gameport-dongle/gameport-dongle.kicad_sch (KiCad schematic)
At the start: 20 parts, among them J1 GAME_IO_DIP16, J2 GAME_IO_DB9, U1 RP2040-Zero, U2 AD5263BRUZ200, U3 74AHCT125

Commit message: Fix empty per-instance Footprint fields in dongle schematic
Symbol instances carried empty Footprint properties that override the
library defaults, so Update-PCB-from-Schematic rejected every part
except C1. Populate each instance's footprint field.

Co-Authored-By: Claude Fable 5 <noreply@anthropic.com>
Claude-Session: https://claude.ai/code/session_01P811gUBbxqALpN1vetBPzG
Parts:
- C2, C3: footprint (none) -> Capacitor_SMD:C_0603_1608Metric
- J1: footprint (none) -> Connector_PinHeader_2.54mm:PinHeader_1x16_P2.54mm_Vertical
- J2: footprint (none) -> Connector_Dsub:DSUB-9_Male_Horizontal_P2.77x2.84mm_EdgePinOffset7.70mm_Housed_MountingHolesOffset9.12mm
- JP1: footprint (none) -> Jumper:SolderJumper-3_P1.3mm_Open_RoundedPad1.0x1.5mm
- R1, R10, R11, R2, R3, R4, R5, R6, R7, R8, R9: footprint (none) -> Resistor_SMD:R_0603_1608Metric
- U1: footprint (none) -> dongle:RP2040-Zero
- U2: footprint (none) -> Package_SO:TSSOP-24_4.4x7.8mm_P0.65mm
- U3: footprint (none) -> Package_SO:SOIC-14_3.9x8.7mm_P1.27mm
Changed lines of the file:
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@@
     (property "Reference" "J1" (at 50.8 101.6 0) (effects (font (size 1.27 1.27))))
     (property "Value" "GAME_IO_DIP16" (at 50.8 104.14 0) (effects (font (size 1.27 1.27))))
-    (property "Footprint" "" (at 50.8 104.14 0) (effects (font (size 1.27 1.27)) hide))
+    (property "Footprint" "Connector_PinHeader_2.54mm:PinHeader_1x16_P2.54mm_Vertical" (at 50.8 104.14 0) (effects (font (size 1.27 1.27)) hide))
     (property "Datasheet" "" (at 50.8 104.14 0) (effects (font (size 1.27 1.27)) hide))
     (pin "1")
@@
     (property "Reference" "J2" (at 50.8 187.96 0) (effects (font (size 1.27 1.27))))
     (property "Value" "GAME_IO_DB9" (at 50.8 190.5 0) (effects (font (size 1.27 1.27))))
-    (property "Footprint" "" (at 50.8 190.5 0) (effects (font (size 1.27 1.27)) hide))
+    (property "Footprint" "Connector_Dsub:DSUB-9_Male_Horizontal_P2.77x2.84mm_EdgePinOffset7.70mm_Housed_MountingHolesOffset9.12mm" (at 50.8 190.5 0) (effects (font (size 1.27 1.27)) hide))
     (property "Datasheet" "" (at 50.8 190.5 0) (effects (font (size 1.27 1.27)) hide))
     (pin "1")
@@
     (property "Reference" "U2" (at 205.74 86.36 0) (effects (font (size 1.27 1.27))))
     (property "Value" "AD5263BRUZ200" (at 205.74 88.9 0) (effects (font (size 1.27 1.27))))
-    (property "Footprint" "" (at 205.74 88.9 0) (effects (font (size 1.27 1.27)) hide))
+    (property "Footprint" "Package_SO:TSSOP-24_4.4x7.8mm_P0.65mm" (at 205.74 88.9 0) (effects (font (size 1.27 1.27)) hide))
     (property "Datasheet" "" (at 205.74 88.9 0) (effects (font (size 1.27 1.27)) hide))
     (pin "VDD")
@@
     (property "Reference" "R1" (at 264.16 86.36 0) (effects (font (size 1.27 1.27))))
     (property "Value" "100R" (at 264.16 88.9 0) (effects (font (size 1.27 1.27))))
-    (property "Footprint" "" (at 264.16 88.9 0) (effects (font (size 1.27 1.27)) hide))
+    (property "Footprint" "Resistor_SMD:R_0603_1608Metric" (at 264.16 88.9 0) (effects (font (size 1.27 1.27)) hide))
     (property "Datasheet" "" (at 264.16 88.9 0) (effects (font (size 1.27 1.27)) hide))
     (pin "1")
@@
     (property "Reference" "R2" (at 281.94000000000005 86.36 0) (effects (font (size 1.27 1.27))))
     (property "Value" "100R" (at 281.94000000000005 88.9 0) (effects (font (size 1.27 1.27))))
-    (property "Footprint" "" (at 281.94000000000005 88.9 0) (effects (font (size 1.27 1.27)) hide))
+    (property "Footprint" "Resistor_SMD:R_0603_1608Metric" (at 281.94000000000005 88.9 0) (effects (font (size 1.27 1.27)) hide))
     (property "Datasheet" "" (at 281.94000000000005 88.9 0) (effects (font (size 1.27 1.27)) hide))
     (pin "1")
@@
     (property "Reference" "R3" (at 299.72 86.36 0) (effects (font (size 1.27 1.27))))
     (property "Value" "100R" (at 299.72 88.9 0) (effects (font (size 1.27 1.27))))
-    (property "Footprint" "" (at 299.72 88.9 0) (effects (font (size 1.27 1.27)) hide))
+    (property "Footprint" "Resistor_SMD:R_0603_1608Metric" (at 299.72 88.9 0) (effects (font (size 1.27 1.27)) hide))
     (property "Datasheet" "" (at 299.72 88.9 0) (effects (font (size 1.27 1.27)) hide))
     (pin "1")
@@
     (property "Reference" "R4" (at 317.5 86.36 0) (effects (font (size 1.27 1.27))))
     (property "Value" "100R" (at 317.5 88.9 0) (effects (font (size 1.27 1.27))))
-    (property "Footprint" "" (at 317.5 88.9 0) (effects (font (size 1.27 1.27)) hide))
+    (property "Footprint" "Resistor_SMD:R_0603_1608Metric" (at 317.5 88.9 0) (effects (font (size 1.27 1.27)) hide))
     (property "Datasheet" "" (at 317.5 88.9 0) (effects (font (size 1.27 1.27)) hide))
     (pin "1")
@@
     (property "Reference" "JP1" (at 205.74 126.99999999999999 0) (effects (font (size 1.27 1.27))))
     (property "Value" "SPI_STRAP" (at 205.74 129.54 0) (effects (font (size 1.27 1.27))))
-    (property "Footprint" "" (at 205.74 129.54 0) (effects (font (size 1.27 1.27)) hide))
+    (property "Footprint" "Jumper:SolderJumper-3_P1.3mm_Open_RoundedPad1.0x1.5mm" (at 205.74 129.54 0) (effects (font (size 1.27 1.27)) hide))
     (property "Datasheet" "" (at 205.74 129.54 0) (effects (font (size 1.27 1.27)) hide))
     (pin "1")
@@
     (property "Reference" "U1" (at 121.92 200.66 0) (effects (font (size 1.27 1.27))))
     (property "Value" "RP2040-Zero" (at 121.92 203.2 0) (effects (font (size 1.27 1.27))))
-    (property "Footprint" "" (at 121.92 203.2 0) (effects (font (size 1.27 1.27)) hide))
+    (property "Footprint" "dongle:RP2040-Zero" (at 121.92 203.2 0) (effects (font (size 1.27 1.27)) hide))
     (property "Datasheet" "" (at 121.92 203.2 0) (effects (font (size 1.27 1.27)) hide))
     (pin "1")
@@
     (property "Reference" "U3" (at 205.74 203.20000000000002 0) (effects (font (size 1.27 1.27))))
     (property "Value" "74AHCT125" (at 205.74 205.74 0) (effects (font (size 1.27 1.27))))
-    (property "Footprint" "" (at 205.74 205.74 0) (effects (font (size 1.27 1.27)) hide))
+    (property "Footprint" "Package_SO:SOIC-14_3.9x8.7mm_P1.27mm" (at 205.74 205.74 0) (effects (font (size 1.27 1.27)) hide))
     (property "Datasheet" "" (at 205.74 205.74 0) (effects (font (size 1.27 1.27)) hide))
     (pin "14")
@@
     (property "Reference" "R5" (at 264.16 149.86 0) (effects (font (size 1.27 1.27))))
     (property "Value" "10k" (at 264.16 152.4 0) (effects (font (size 1.27 1.27))))
-    (property "Footprint" "" (at 264.16 152.4 0) (effects (font (size 1.27 1.27)) hide))
+    (property "Footprint" "Resistor_SMD:R_0603_1608Metric" (at 264.16 152.4 0) (effects (font (size 1.27 1.27)) hide))
     (property "Datasheet" "" (at 264.16 152.4 0) (effects (font (size 1.27 1.27)) hide))
     (pin "1")
@@
     (property "Reference" "R6" (at 281.94000000000005 149.86 0) (effects (font (size 1.27 1.27))))
     (property "Value" "10k" (at 281.94000000000005 152.4 0) (effects (font (size 1.27 1.27))))
-    (property "Footprint" "" (at 281.94000000000005 152.4 0) (effects (font (size 1.27 1.27)) hide))
+    (property "Footprint" "Resistor_SMD:R_0603_1608Metric" (at 281.94000000000005 152.4 0) (effects (font (size 1.27 1.27)) hide))
     (property "Datasheet" "" (at 281.94000000000005 152.4 0) (effects (font (size 1.27 1.27)) hide))
     (pin "1")
@@
     (property "Reference" "R7" (at 299.72 149.86 0) (effects (font (size 1.27 1.27))))
     (property "Value" "10k" (at 299.72 152.4 0) (effects (font (size 1.27 1.27))))
-    (property "Footprint" "" (at 299.72 152.4 0) (effects (font (size 1.27 1.27)) hide))
+    (property "Footprint" "Resistor_SMD:R_0603_1608Metric" (at 299.72 152.4 0) (effects (font (size 1.27 1.27)) hide))
     (property "Datasheet" "" (at 299.72 152.4 0) (effects (font (size 1.27 1.27)) hide))
     (pin "1")
@@
     (property "Reference" "R8" (at 317.5 149.86 0) (effects (font (size 1.27 1.27))))
     (property "Value" "10k" (at 317.5 152.4 0) (effects (font (size 1.27 1.27))))
-    (property "Footprint" "" (at 317.5 152.4 0) (effects (font (size 1.27 1.27)) hide))
+    (property "Footprint" "Resistor_SMD:R_0603_1608Metric" (at 317.5 152.4 0) (effects (font (size 1.27 1.27)) hide))
     (property "Datasheet" "" (at 317.5 152.4 0) (effects (font (size 1.27 1.27)) hide))
     (pin "1")
@@
     (property "Reference" "R9" (at 264.16 200.66 0) (effects (font (size 1.27 1.27))))
     (property "Value" "560R" (at 264.16 203.2 0) (effects (font (size 1.27 1.27))))
-    (property "Footprint" "" (at 264.16 203.2 0) (effects (font (size 1.27 1.27)) hide))
+    (property "Footprint" "Resistor_SMD:R_0603_1608Metric" (at 264.16 203.2 0) (effects (font (size 1.27 1.27)) hide))
     (property "Datasheet" "" (at 264.16 203.2 0) (effects (font (size 1.27 1.27)) hide))
     (pin "1")
@@
     (property "Reference" "R10" (at 281.94000000000005 200.66 0) (effects (font (size 1.27 1.27))))
     (property "Value" "560R" (at 281.94000000000005 203.2 0) (effects (font (size 1.27 1.27))))
-    (property "Footprint" "" (at 281.94000000000005 203.2 0) (effects (font (size 1.27 1.27)) hide))
+    (property "Footprint" "Resistor_SMD:R_0603_1608Metric" (at 281.94000000000005 203.2 0) (effects (font (size 1.27 1.27)) hide))
     (property "Datasheet" "" (at 281.94000000000005 203.2 0) (effects (font (size 1.27 1.27)) hide))
     (pin "1")
@@
     (property "Reference" "R11" (at 299.72 200.66 0) (effects (font (size 1.27 1.27))))
     (property "Value" "560R" (at 299.72 203.2 0) (effects (font (size 1.27 1.27))))
-    (property "Footprint" "" (at 299.72 203.2 0) (effects (font (size 1.27 1.27)) hide))
+    (property "Footprint" "Resistor_SMD:R_0603_1608Metric" (at 299.72 203.2 0) (effects (font (size 1.27 1.27)) hide))
     (property "Datasheet" "" (at 299.72 203.2 0) (effects (font (size 1.27 1.27)) hide))
     (pin "1")
@@
     (property "Reference" "C2" (at 345.44 200.66 0) (effects (font (size 1.27 1.27))))
     (property "Value" "100nF" (at 345.44 203.2 0) (effects (font (size 1.27 1.27))))
-    (property "Footprint" "" (at 345.44 203.2 0) (effects (font (size 1.27 1.27)) hide))
+    (property "Footprint" "Capacitor_SMD:C_0603_1608Metric" (at 345.44 203.2 0) (effects (font (size 1.27 1.27)) hide))
     (property "Datasheet" "" (at 345.44 203.2 0) (effects (font (size 1.27 1.27)) hide))
     (pin "1")
@@
     (property "Reference" "C3" (at 360.68 200.66 0) (effects (font (size 1.27 1.27))))
     (property "Value" "100nF" (at 360.68 203.2 0) (effects (font (size 1.27 1.27))))
-    (property "Footprint" "" (at 360.68 203.2 0) (effects (font (size 1.27 1.27)) hide))
+    (property "Footprint" "Capacitor_SMD:C_0603_1608Metric" (at 360.68 203.2 0) (effects (font (size 1.27 1.27)) hide))
     (property "Datasheet" "" (at 360.68 203.2 0) (effects (font (size 1.27 1.27)) hide))
     (pin "1")
